Commit message: package name bug fixes

File: xacro/depthcam.xacro (robot description, xacro)
@@ -1,5 +1,5 @@
 <?xml version="1.0"?>
 <robot xmlns:xacro="http://www.ros.org/wiki/xacro">
-  <xacro:include filename="$(find realsense_435_description)/xacro/inertia_calc.xacro"/>
+  <xacro:include filename="$(find realsense435_description)/xacro/inertia_calc.xacro"/>
   <!-- INTEL REALSENSE D435 -->
   <xacro:macro name="realsense_d435" params="sensor_name parent_link *origin rate">
@@ -31,5 +31,5 @@
         <origin xyz="${d435_cam_mount_from_center_offset} ${-d435_cam_depth_py} 0" rpy="${pi/2} 0 ${pi/2}"/>
         <geometry>
-          <mesh filename="package://realsense_435_description/meshes/realsense_d435.stl" />
+          <mesh filename="package://realsense435_description/meshes/realsense_d435.stl" />
         </geometry>
       </visual>

File: xacro/depthcam_with_gazebo.xacro (robot description, xacro)
@@ -1,5 +1,5 @@
 <?xml version="1.0"?>
 <robot xmlns:xacro="http://www.ros.org/wiki/xacro">
-  <xacro:include filename="$(find realsense_ros_gazebo)/xacro/inertia_calc.xacro"/>
+  <xacro:include filename="$(find realsense435_description)/xacro/inertia_calc.xacro"/>
   <!-- INTEL REALSENSE D435 -->
   <xacro:macro name="realsense_d435" params="sensor_name parent_link *origin rate">
@@ -31,5 +31,5 @@
         <origin xyz="${d435_cam_mount_from_center_offset} ${-d435_cam_depth_py} 0" rpy="${pi/2} 0 ${pi/2}"/>
         <geometry>
-          <mesh filename="package://realsense_ros_gazebo/meshes/realsense_d435.stl" />
+          <mesh filename="package://realsense435_description/meshes/realsense_d435.stl" />
         </geometry>
       </visual>
